File: P01_Hydroponics/Sensors_sch.kicad_sch (KiCad schematic)
At the start: 9 parts, among them J2 JST_PH_3P_TEMP, J3 JST_PH_3P_FLOW, J4 JST_PH_3P_WLS1, J5 JST_PH_4P_WLS0, J6 JST_PH_2P_PUMP, Q2 NMOS

Commit message: New version
Modified PD sink controller, and added 3v3 and 5V DC-DC buck converters
Parts:
- R16, R17: symbol Device:R -> Device:R_Small
Connections:
- net GND: no longer R17.2
- net PWM1: no longer R16.1
- now unconnected: Q2.2 (G), R16.2, R17.1
Changed lines of the file:
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@@
 	)
 	(symbol
-		(lib_id "Device:R")
+		(lib_id "Device:R_Small")
 		(at 35.56 48.26 0)
 		(unit 1)
@@
 		)
 		(property "Footprint" ""
-			(at 33.782 48.26 90)
-			(effects
-				(font
-					(size 1.27 1.27)
-				)
-				(hide yes)
-			)
-		)
-		(property "Datasheet" "~"
 			(at 35.56 48.26 0)
 			(effects
@@
 			)
 		)
-		(property "Description" "Resistor"
+		(property "Datasheet" "~"
+			(at 35.56 48.26 0)
+			(effects
+				(font
+					(size 1.27 1.27)
+				)
+				(hide yes)
+			)
+		)
+		(property "Description" "Resistor, small symbol"
 			(at 35.56 48.26 0)
 			(effects
@@
 		(dnp no)
 		(fields_autoplaced yes)
-		(property "Reference" "#PWR051"
+		(property "Reference" "#PWR052"
 			(at 45.72 60.96 0)
 			(effects
@@
 			(project ""
 				(path "/f251d969-db3d-42b0-b168-8992c4b2bbf4/d0dfc5ef-a144-4c79-b9fc-fc1612b2e1ba"
-					(reference "#PWR051")
+					(reference "#PWR052")
 					(unit 1)
 				)
@@
 	)
 	(symbol
-		(lib_id "Device:R")
+		(lib_id "Device:R_Small")
 		(at 29.21 41.91 90)
 		(unit 1)
@@
 		(fields_autoplaced yes)
 		(property "Reference" "R16"
-			(at 29.21 35.56 90)
+			(at 29.21 36.83 90)
 			(effects
 				(font
@@
 		)
 		(property "Value" "R"
-			(at 29.21 38.1 90)
-			(effects
-				(font
-					(size 1.27 1.27)
-				)
-			)
-		)
-		(property "Footprint" ""
-			(at 29.21 43.688 90)
-			(effects
-				(font
-					(size 1.27 1.27)
-				)
-				(hide yes)
-			)
-		)
-		(property "Datasheet" "~"
+			(at 29.21 39.37 90)
+			(effects
+				(font
+					(size 1.27 1.27)
+				)
+			)
+		)
+		(property "Footprint" ""
 			(at 29.21 41.91 0)
 			(effects
@@
 			)
 		)
-		(property "Description" "Resistor"
+		(property "Datasheet" "~"
 			(at 29.21 41.91 0)
 			(effects
+				(font
+					(size 1.27 1.27)
+				)
+				(hide yes)
+			)
+		)
+		(property "Description" "Resistor, small symbol"
+			(at 29.21 41.91 0)
+			(effects
