File: P01_Hydroponics/_autosave-Battery_charger_sch.kicad_sch (KiCad schematic)
At the start: 39 parts, among them Q5 PMOS, U3 TPSM33625RDNR, U4 TPSM33625RDNR, U5 BQ25306

Commit message: Need review
Please review the schematics.
Parts:
- R27: value `? -> R_Small
- R28: value ? -> R_Small
Connections:
- net REGN: now also RT1.2; no longer RT1.1
- net at RT2.2, TH2.1, U5.7 (TS): now also RT1.1; no longer RT1.2
- net +3.3V renamed +3V3
- net +5V renamed +5VP
- net ICH1 renamed PB0
- net ICH2 renamed PB1
Other:
- note removed: "Protection/ gauging?"
- moved on the sheet: BT1, C25, C26, C27, C28, C29, C30, C31, C32, C33, C34, C35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
