File: P01_Hydroponics/_autosave-Power.kicad_sch (KiCad schematic)
At the start: 39 parts, among them Q5 PMOS, U3 TPSM33625RDNR, U4 TPSM33625RDNR, U5 BQ25306

Commit message: Need review
Please review the schematics.
Other:
- note removed: "Protection/ gauging?"
Changed lines of the file:
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@@
 	)
 	(bus_entry
-		(at 274.32 21.59)
+		(at 273.05 20.32)
 		(size -2.54 2.54)
 		(stroke
@@
 	)
 	(bus_entry
-		(at 274.32 24.13)
+		(at 273.05 22.86)
 		(size -2.54 2.54)
 		(stroke
@@
 	(bus
 		(pts
-			(xy 274.32 20.32) (xy 274.32 21.59)
+			(xy 273.05 19.05) (xy 273.05 20.32)
 		)
 		(stroke
@@
 	(wire
 		(pts
-			(xy 262.89 26.67) (xy 271.78 26.67)
+			(xy 261.62 25.4) (xy 270.51 25.4)
 		)
 		(stroke
@@
 	(bus
 		(pts
-			(xy 276.86 20.32) (xy 274.32 20.32)
+			(xy 275.59 19.05) (xy 273.05 19.05)
 		)
 		(stroke
@@
 	(bus
 		(pts
-			(xy 274.32 24.13) (xy 274.32 26.67)
+			(xy 273.05 22.86) (xy 273.05 25.4)
 		)
 		(stroke
@@
 	(bus
 		(pts
-			(xy 274.32 21.59) (xy 274.32 24.13)
+			(xy 273.05 20.32) (xy 273.05 22.86)
 		)
 		(stroke
@@
 	(wire
 		(pts
-			(xy 123.19 36.83) (xy 127 36.83)
-		)
-		(stroke
-			(width 0)
-			(type default)
-		)
-	)
-	(wire
-		(pts
 			(xy 104.14 67.31) (xy 104.14 72.39)
 		)
@@
 	(wire
 		(pts
-			(xy 262.89 24.13) (xy 271.78 24.13)
+			(xy 261.62 22.86) (xy 270.51 22.86)
 		)
 		(stroke
@@
 		(start 43.18 17.78)
 		(end 256.54 128.27)
-		(stroke
-			(width 0)
-			(type default)
-		)
-		(fill
-			(type none)
-		)
-	)
-	(rectangle
-		(start 171.45 71.12)
-		(end 238.76 111.76)
 		(stroke
 			(width 0)
@@
 			)
 			(justify left top)
-		)
-	)
-	(text "Protection/ gauging?"
-		(exclude_from_sim no)
-		(at 206.248 91.186 0)
-		(effects
-			(font
-				(size 1.27 1.27)
-			)
 		)
 	)
@@
 	)
 	(label "ICH2"
-		(at 262.89 26.67 0)
+		(at 261.62 25.4 0)
 		(fields_autoplaced yes)
 		(effects
@@
 	)
 	(label "ICH1"
-		(at 262.89 24.13 0)
+		(at 261.62 22.86 0)
 		(fields_autoplaced yes)
 		(effects
@@
 	(hierarchical_label "{IO}"
 		(shape input)
-		(at 276.86 20.32 0)
+		(at 275.59 19.05 0)
 		(fields_autoplaced yes)
 		(effects
