File: P01_Hydroponics/USB-Type C PD_sch.kicad_sch (KiCad schematic)
At the start: 42 parts, among them J7 USB_C_Receptacle_USB2.0_16P, Q3 NMOS, Q4 NMOS, Q5 PMOS, U3 TPSM33625RDNR, U4 TPSM33625RDNR

Commit message: Retry
bla bla
Parts:
- removed C25, C26, C31, C32: 22uF, symbol Device:C_Small
- removed C27, C28, C29, C30, C33: 4.7uF, symbol Device:C_Small
- removed D9: Dual Schottky common anode, symbol Device:D_Schottky_Dual_CommonAnode_AKK_Parallel
- removed Q5: PMOS, symbol Simulation_SPICE:PMOS
- removed R27: 23.2K, symbol Device:R_Small
- removed R28, R34: 10K, symbol Device:R_Small
- removed R29, R30: R_Small, symbol Device:R_Small
- removed R31: 19.8K, symbol Device:R_Small
- removed R33: 40.2K, symbol Device:R_Small
- removed U3, U4: TPSM33625RDNR, symbol DC-DC-Converter:TPSM33625RDNR
Other:
- moved on the sheet: C20, C21, C22, C23, C24, D6, D7, D8, J7, Q3, Q4, R18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

Commit message: Need review
Please review the schematics.
Parts:
- removed Q3, Q4: NMOS, symbol Simulation_SPICE:NMOS
- added Q3, Q4: BSS138, Package_TO_SOT_SMD:SOT-23, symbol Transistor_FET:BSS138
- added Q8, Q9: DMN3008SFG, Package_SON:Diodes_PowerDI3333-8, symbol Transistor_FET:DMN3008SFG
- added R34, R35, R36, R37: 10k, symbol Device:R_Small
- R23: value 10R -> 0R
- U2: value ~ -> AP33772S; footprint (none) -> Package_DFN_QFN:QFN-24-1EP_4x4mm_P0.5mm_EP2.7x2.7mm
Connections:
- net SCL_5V: now also Q3.3 (D), R37.2
- net SDA_5V: now also Q4.3 (D), R35.2
- net VS: now also Q8.1 (S), Q8.2 (S), Q8.3 (S)
- net VSYS: now also Q9.1 (S), Q9.2 (S), Q9.3 (S)
- net at R23.1: now also Q8.4 (G), Q9.4 (G)
- net V5V: now reaches C20.2, U2.20 (V5V)
- net V5V: now also R35.1, R37.1
- new net: Q8.5 (D), Q9.5 (D)
- new net +3.3V: Q3.1 (G), Q4.1 (G), R34.1, R36.1
- new net I2C_SCL: Q3.2 (S), R36.2
- new net I2C_SDA: Q4.2 (S), R34.2
Other:
- note added: "AP33772S I2C PD sink controller"
- note added: "Level shifter"
- moved on the sheet: C20, C21, C22, C23, C24, D6, D7, D8, J7, R18, R19, R20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

Commit message: Need review
Updated:
STD14 to tag connect.
Added most footprints.
Change crystal to oscillator for ESP32
Rearrange radio controller schematic.
Added NOR flash.
Added USB-C connector for ESP32
Parts:
- removed C22: 0.1uF, symbol Device:C_Small
- removed C23, C24: 10uF, symbol Device:C_Small
- added C17, C19: 10uF/25VDC, Capacitor_SMD:C_0603_1608Metric_Pad1.08x0.95mm_HandSolder, symbol Device:C_Small
- added C18: 1uF/10VDC, Capacitor_SMD:C_0603_1608Metric_Pad1.08x0.95mm_HandSolder, symbol Device:C_Small
- C20: value 1uF -> 0.1uF/10VDC; footprint (none) -> Capacitor_SMD:C_0603_1608Metric_Pad1.08x0.95mm_HandSolder; Dielectric (none) -> X7R
- C21: value 0.1uF -> 0.1uF/10VDC; footprint (none) -> Capacitor_SMD:C_0603_1608Metric_Pad1.08x0.95mm_HandSolder; Dielectric (none) -> X7R
- D7: renamed from D8; footprint (none) -> LED_SMD:LED_0603_1608Metric_Pad1.05x0.95mm_HandSolder
- D8: renamed from D7; footprint (none) -> LED_SMD:LED_0603_1608Metric_Pad1.05x0.95mm_HandSolder
- R20: renamed from R21; footprint (none) -> Resistor_SMD:R_0603_1608Metric_Pad0.98x0.95mm_HandSolder
- R21: renamed from R20; footprint (none) -> Resistor_SMD:R_0603_1608Metric_Pad0.98x0.95mm_HandSolder
- R22: renamed from R19; footprint (none) -> Resistor_SMD:R_0603_1608Metric_Pad0.98x0.95mm_HandSolder
- R23: renamed from R18; footprint (none) -> Resistor_SMD:R_0603_1608Metric_Pad0.98x0.95mm_HandSolder
- R24: renamed from R26; footprint (none) -> Resistor_SMD:R_0603_1608Metric_Pad0.98x0.95mm_HandSolder
- R25: renamed from R22; footprint (none) -> Resistor_SMD:R_1210_3225Metric_Pad1.30x2.65mm_HandSolder
- R26: renamed from R25; footprint (none) -> Resistor_SMD:R_0603_1608Metric_Pad0.98x0.95mm_HandSolder
- R27: renamed from R23; footprint (none) -> Resistor_SMD:R_0603_1608Metric_Pad0.98x0.95mm_HandSolder
- R28: renamed from R24; footprint (none) -> Resistor_SMD:R_0603_1608Metric_Pad0.98x0.95mm_HandSolder
- R29: renamed from R34; footprint (none) -> Resistor_SMD:R_0603_1608Metric_Pad0.98x0.95mm_HandSolder
- R30: renamed from R36; footprint (none) -> Resistor_SMD:R_0603_1608Metric_Pad0.98x0.95mm_HandSolder
- R31: renamed from R35; footprint (none) -> Resistor_SMD:R_0603_1608Metric_Pad0.98x0.95mm_HandSolder
- R32: renamed from R37; footprint (none) -> Resistor_SMD:R_0603_1608Metric_Pad0.98x0.95mm_HandSolder
- TH1: footprint (none) -> Resistor_SMD:R_0603_1608Metric_Pad0.98x0.95mm_HandSolder
- renumbered J7 to J8, Q8 to Q5, Q9 to Q6, Q4 to Q7, Q3 to Q8, U2 to U3
Connections:
- net GND: now also C17.1, C18.1, C19.1
- net V5V: now also C18.2; no longer C20.2
- net VBUS: now also C17.2
- net VSYS: now also C19.2
- net at U3.12 (V18): now also C20.2; no longer C21.2
- net at U3.15 (IFB): now also C21.2
