File: P01_Hydroponics/User.Interface_sch.kicad_sch (KiCad schematic)
At the start: 11 parts, among them Q1 NMOS

Commit message: New version
Modified PD sink controller, and added 3v3 and 5V DC-DC buck converters
Parts:
- C16, C17, C18, C19: symbol Device:C -> Device:C_Small
- R14, R15: symbol Device:R -> Device:R_Small

Commit message: Need review
Please review the schematics.
Changed lines of the file:
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@@
 		(color 0 0 0 0)
 	)
+	(bus_entry
+		(at 200.66 60.96)
+		(size -2.54 2.54)
+		(stroke
+			(width 0)
+			(type default)
+		)
+	)
+	(bus
+		(pts
+			(xy 204.47 59.69) (xy 200.66 59.69)
+		)
+		(stroke
+			(width 0)
+			(type default)
+		)
+	)
 	(wire
 		(pts
@@
 		)
 	)
+	(bus
+		(pts
+			(xy 200.66 59.69) (xy 200.66 60.96)
+		)
+		(stroke
+			(width 0)
+			(type default)
+		)
+	)
 	(wire
 		(pts
@@
 		)
 	)
+	(bus
+		(pts
+			(xy 200.66 60.96) (xy 200.66 63.5)
+		)
+		(stroke
+			(width 0)
+			(type default)
+		)
+	)
 	(wire
 		(pts
@@
 	(wire
 		(pts
+			(xy 187.96 63.5) (xy 198.12 63.5)
+		)
+		(stroke
+			(width 0)
+			(type default)
+		)
+	)
+	(wire
+		(pts
 			(xy 172.72 93.98) (xy 184.15 93.98)
 		)
@@
 	(wire
 		(pts
-			(xy 199.39 93.98) (xy 210.82 93.98)
+			(xy 199.39 93.98) (xy 204.47 93.98)
 		)
 		(stroke
@@
 		)
 	)
-	(label "DIN"
-		(at 96.52 93.98 0)
-		(fields_autoplaced yes)
-		(effects
-			(font
-				(size 1.27 1.27)
-			)
-			(justify left bottom)
-		)
-	)
 	(label "LED_EN"
 		(at 138.43 76.2 180)
@@
 		)
 	)
+	(label "LED_EN"
+		(at 187.96 63.5 0)
+		(fields_autoplaced yes)
+		(effects
+			(font
+				(size 1.27 1.27)
+			)
+			(justify left bottom)
+		)
+	)
 	(label "V_led"
 		(at 116.84 83.82 0)
@@
 		)
 	)
-	(label "DOUT"
-		(at 210.82 93.98 180)
-		(fields_autoplaced yes)
-		(effects
-			(font
-				(size 1.27 1.27)
-			)
-			(justify right bottom)
-		)
-	)
+	(hierarchical_label "DIN"
+		(shape input)
+		(at 96.52 93.98 180)
+		(fields_autoplaced yes)
+		(effects
+			(font
+				(size 1.27 1.27)
+			)
+			(justify right)
+		)
+	)
+	(hierarchical_label "DOUT"
+		(shape output)
+		(at 204.47 93.98 0)
+		(fields_autoplaced yes)
+		(effects
+			(font
+				(size 1.27 1.27)
+			)
+			(justify left)
+		)
+	)
+	(hierarchical_label "{IO}"
+		(shape input)
+		(at 204.47 59.69 0)
+		(fields_autoplaced yes)
+		(effects
+			(font
+				(size 1.27 1.27)
+			)
+			(justify left)
+		)
+	)

Commit message: Need review
Updated:
STD14 to tag connect.
Added most footprints.
Change crystal to oscillator for ESP32
Rearrange radio controller schematic.
Added NOR flash.
Added USB-C connector for ESP32
Parts:
- removed C17, C18, C19: 0.1uF, symbol Device:C_Small
- removed Q1: NMOS, symbol Simulation_SPICE:NMOS
- added C13, C14, C15: 0.1uF/10VDC, Capacitor_SMD:C_0603_1608Metric_Pad1.08x0.95mm_HandSolder, symbol Device:C_Small
- added Q1: SQ2337CES-T1_GE3, Package_TO_SOT_SMD:SOT-23-3, symbol Simulation_SPICE:PMOS
- C16: value 0.1uF -> 0.1uF/10VDC; footprint (none) -> Capacitor_SMD:C_0603_1608Metric_Pad1.08x0.95mm_HandSolder; Dielectric (none) -> X7R
- R11: renamed from R15; footprint (none) -> Resistor_SMD:R_0603_1608Metric_Pad0.98x0.95mm_HandSolder
- R12: renamed from R14; footprint (none) -> Resistor_SMD:R_0603_1608Metric_Pad0.98x0.95mm_HandSolder
Connections:
- net +3.3V: now also Q1.1 (D)
- net GND: now also C13.1, C14.1, C15.1
- net V_led: now also C13.2, C14.2, C15.2, Q1.3 (S)
- net at R11.1: now also Q1.2 (G)
